File: vic2020mainboard/Vic2020mainboard.kicad_pcb (KiCad board)
At the start: 2 copper layers, 357.8 x 124.5 mm, 142 parts, among them J1 A15 KERNAL/BASIC SELECT, J10 5v Regulated, J11 Conn_02x08_Odd_Even, J12 Conn_02x22_Row_Letter_First, J13 IEC Port, J14 Joystick 1, J2 A14 Kernel/Basic Select, J3 FONT SELECT, J4 Chroma Disconnect, J5 SVIDEO Out, J6 Audio Out, J7 Video Out, J8 Keyboard, J9 LED, Q1 2sc1959, Q2 2SC1815, SW1 RAM ENABLE, SW3 Expansion Port, U1 7402, U10 74LS133, U11 74LS02, U12 AS6C1008-55PCN, U13 27512, U14 74LS245, U15 74LS245, U16 74LS245, U17 AS6C1008-55PCN, U18 74LS245, U19 2764, U2 74LS138, U20 6560, U21 W65C22NxP, U22 W65C22NxP, U23 74LS245, U24 74ALS32, U3 LM555, U4 7406, U5 74LS133, U6 74LS138, U7 W65C02SxP, U8 74LS00, U9 74LS04, Y1 Crystal

Commit message: Allow for edge connectors with larger pins on J12.
Parts:
- moved J12 90.9 mm to (383.6, 98.7)
Routing:
- net D7: track 462.0 -> 452.1 mm, vias 7 -> 8
- net A7: track 452.6 -> 446.5 mm, vias 4 -> 5
- net CBLK1: track 81.0 -> 84.2 mm
- net IO2: track 178.8 -> 181.6 mm
- net D6: track 495.1 -> 497.7 mm
- net BLK2: track 181.8 -> 184.1 mm
- net A6: track 421.5 -> 423.4 mm
- net D0: track 550.7 -> 552.5 mm
- net D1: track 459.3 -> 461.1 mm
- net A2: track 432.0 -> 433.6 mm
- net CBLK2: track 78.7 -> 80.3 mm
- net A1: track 403.5 -> 404.8 mm
- net A4: track 471.0 -> 471.8 mm
- net A0: track 463.2 -> 464.0 mm
- net A5: track 489.8 -> 490.6 mm
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Other:
- net class Default removed
- net class GROUND removed
- net class POWER removed
